File: LSA Design Task/LSA Design.kicad_pcb (KiCad board)
At the start: 2 copper layers, 61 x 33 mm, 18 parts, among them J1 Conn_02x05_Odd_Even, P1 D_Photo, P2 D_Photo, P3 D_Photo, P4 D_Photo, U1 LM324

Commit message: vault backup: 2022-09-01 12:03:59
Routing:
- net GND: track 158.1 -> 1.32 mm, vias 2 -> 0
- added copper zone on B.Cu, net GND
Changed lines of the file:
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@@
   (segment (start 97 88) (end 97 84.5) (width 0.2) (layer "B.Cu") (net 2))
   (segment (start 96.08 83.58) (end 94.5 83.58) (width 0.2) (layer "B.Cu") (net 2))
-  (segment (start 103.225 94.5) (end 89.225 94.5) (width 0.4) (layer "F.Cu") (net 3))
-  (segment (start 123.225 96.5) (end 124.907154 94.817846) (width 0.4) (layer "F.Cu") (net 3))
-  (segment (start 141.225 95.725) (end 139 93.5) (width 0.4) (layer "F.Cu") (net 3))
-  (segment (start 94.5 73.42) (end 101 73.42) (width 0.4) (layer "F.Cu") (net 3))
-  (segment (start 92 91) (end 92 90.5) (width 0.4) (layer "F.Cu") (net 3))
-  (segment (start 111.67 72.9975) (end 110.42 71.7475) (width 0.4) (layer "F.Cu") (net 3))
-  (segment (start 139 93.5) (end 139 90.5) (width 0.4) (layer "F.Cu") (net 3))
-  (segment (start 89.225 94.5) (end 87.225 96.5) (width 0.4) (layer "F.Cu") (net 3))
-  (segment (start 87.225 95.775) (end 92 91) (width 0.4) (layer "F.Cu") (net 3))
-  (segment (start 141.225 96.5) (end 141.225 95.725) (width 0.4) (layer "F.Cu") (net 3))
-  (segment (start 130.0775 72.9975) (end 111.67 72.9975) (width 0.4) (layer "F.Cu") (net 3))
   (segment (start 87.225 96.5) (end 87.225 95.775) (width 0.4) (layer "F.Cu") (net 3))
-  (segment (start 124.907154 94.817846) (end 139.542846 94.817846) (width 0.4) (layer "F.Cu") (net 3))
   (segment (start 130.5 73.42) (end 130.0775 72.9975) (width 0.4) (layer "F.Cu") (net 3))
-  (segment (start 108.7475 73.42) (end 110.42 71.7475) (width 0.4) (layer "F.Cu") (net 3))
-  (segment (start 101 73.42) (end 108.7475 73.42) (width 0.4) (layer "F.Cu") (net 3))
-  (segment (start 105.225 96.5) (end 103.225 94.5) (width 0.4) (layer "F.Cu") (net 3))
-  (segment (start 139.542846 94.817846) (end 141.225 96.5) (width 0.4) (layer "F.Cu") (net 3))
-  (segment (start 136.5 73.42) (end 130.5 73.42) (width 0.4) (layer "F.Cu") (net 3))
-  (via (at 139 90.5) (size 0.8) (drill 0.4) (layers "F.Cu" "B.Cu") (net 3))
-  (via (at 92 90.5) (size 0.8) (drill 0.4) (layers "F.Cu" "B.Cu") (net 3))
-  (segment (start 114.11 71.11) (end 113.5 70.5) (width 0.2) (layer "B.Cu") (net 3))
-  (segment (start 116 85.53) (end 116 76.653846) (width 0.2) (layer "B.Cu") (net 3))
-  (segment (start 113.5 70.5) (end 111.6675 70.5) (width 0.2) (layer "B.Cu") (net 3))
-  (segment (start 119.47 89) (end 116 85.53) (width 0.2) (layer "B.Cu") (net 3))
-  (segment (start 92 90.5) (end 92 75.92) (width 0.4) (layer "B.Cu") (net 3))
-  (segment (start 92 75.92) (end 94.5 73.42) (width 0.4) (layer "B.Cu") (net 3))
-  (segment (start 111.6675 70.5) (end 110.42 71.7475) (width 0.2) (layer "B.Cu") (net 3))
-  (segment (start 139 75.92) (end 136.5 73.42) (width 0.4) (layer "B.Cu") (net 3))
-  (segment (start 139 90.5) (end 139 75.92) (width 0.4) (layer "B.Cu") (net 3))
-  (segment (start 114.11 74.763846) (end 114.11 71.11) (width 0.2) (layer "B.Cu") (net 3))
-  (segment (start 116 76.653846) (end 114.11 74.763846) (width 0.2) (layer "B.Cu") (net 3))
   (segment (start 104.5 95) (end 107 95) (width 0.2) (layer "F.Cu") (net 4))
   (segment (start 103 89.5) (end 103 93.5) (width 0.2) (layer "F.Cu") (net 4))
@@
   (segment (start 131.5 95) (end 131.5 88.42) (width 0.2) (layer "B.Cu") (net 18))
   (segment (start 131 95.5) (end 131.5 95) (width 0.2) (layer "B.Cu") (net 18))
+  (zone (net 3) (net_name "GND") (layer "B.Cu") (hatch edge 0.508)
+    (connect_pads (clearance 0.508))
+    (min_thickness 0.254) (filled_areas_thickness no)
+    (fill yes (thermal_gap 0.508) (thermal_bridge_width 0.508))
+    (polygon
+      (pts
+        (xy 146.5 100.5)
+        (xy 84.5 100.5)
+        (xy 84.5 66.5)
+        (xy 146.5 66.5)
+      )
+    )
+  )
 )
