File: Latest/Latest.kicad_pcb (KiCad board)
At the start: 2 copper layers, 80 x 64 mm, 0 parts

Commit message: vault backup: 2022-09-11 00:08:13
Parts:
- added C1: 22uF, Capacitor_SMD:C_0805_2012Metric, F.Cu at (250.2, 86.2)
- added C2: 22uF, Capacitor_SMD:C_0805_2012Metric, F.Cu at (245.8, 86.2)
- added D2: LED, LED_SMD:LED_1206_3216Metric, F.Cu at (235.7, 73.2)
- added D3: LED, LED_SMD:LED_1206_3216Metric, F.Cu at (220.8, 123.5)
- added D4: LED, LED_SMD:LED_1206_3216Metric, F.Cu at (230.1, 73.2)
- added D5: LED, LED_SMD:LED_1206_3216Metric, F.Cu at (247.0, 73.2)
- added D6: LED, LED_SMD:LED_1206_3216Metric, F.Cu at (241.3, 73.2)
- added J1: Conn_01x19_Male, Connector_PinHeader_2.54mm:PinHeader_1x19_P2.54mm_Vertical, F.Cu at (224.9, 73.8)
- added J2: Conn_01x19_Male, Connector_PinHeader_2.54mm:PinHeader_1x19_P2.54mm_Vertical, F.Cu at (220.2, 73.8)
- added JP1: SolderJumper_2_Open, Jumper:SolderJumper-2_P1.3mm_Open_Pad1.0x1.5mm, F.Cu at (254.7, 86.4)
- added R1: 2.2K, Resistor_SMD:R_1206_3216Metric, F.Cu at (246.8, 79.8)
- added R10: R, Resistor_SMD:R_1206_3216Metric, F.Cu at (258.1, 79.7)
- added R11: R, Resistor_SMD:R_1206_3216Metric, F.Cu at (241.2, 79.8)
- added R12: R, Resistor_SMD:R_1206_3216Metric, F.Cu at (235.6, 79.8)
- added R13: R, Resistor_SMD:R_1206_3216Metric, F.Cu at (258.2, 73.1)
- added R14: R, Resistor_SMD:R_1206_3216Metric, F.Cu at (258.2, 76.4)
- added R15: R, Resistor_SMD:R_1206_3216Metric, F.Cu at (246.8, 76.5)
- added R18: R, Resistor_SMD:R_1206_3216Metric, F.Cu at (235.6, 83.1)
- added R19: R, Resistor_SMD:R_1206_3216Metric, F.Cu at (235.6, 76.5)
- added R2: R, Resistor_SMD:R_1206_3216Metric, F.Cu at (263.7, 79.7)
- added R20: R, Resistor_SMD:R_1206_3216Metric, F.Cu at (252.6, 73.1)
- added R21: R, Resistor_SMD:R_1206_3216Metric, F.Cu at (230.0, 79.7)
- added R22: R, Resistor_SMD:R_1206_3216Metric, F.Cu at (252.4, 83.0)
- added R23: R, Resistor_SMD:R_1206_3216Metric, F.Cu at (263.7, 83.0)
- added R24: R, Resistor_SMD:R_1206_3216Metric, F.Cu at (241.2, 83.1)
- added R25: R, Resistor_SMD:R_1206_3216Metric, F.Cu at (252.6, 76.4)
- added R26: R, Resistor_SMD:R_1206_3216Metric, F.Cu at (246.8, 83.1)
- added R3: R, Resistor_SMD:R_1206_3216Metric, F.Cu at (263.8, 73.1)
- added R4: R, Resistor_SMD:R_1206_3216Metric, F.Cu at (241.2, 76.5)
- added R5: R, Resistor_SMD:R_1206_3216Metric, F.Cu at (230.0, 86.3)
- added R6: R, Resistor_SMD:R_1206_3216Metric, F.Cu at (263.8, 76.4)
- added R7: R, Resistor_SMD:R_1206_3216Metric, F.Cu at (252.4, 79.7)
- added R8: R, Resistor_SMD:R_1206_3216Metric, F.Cu at (235.6, 86.4)
- added R9: R, Resistor_SMD:R_1206_3216Metric, F.Cu at (258.1, 83.0)
- added U2: MT3608, Package_TO_SOT_SMD:SOT-23-6, F.Cu at (241.0, 87.0)
Other:
- board size 80 x 64 mm -> 80 x 62.5 mm

Commit message: vault backup: 2022-10-02 12:01:12
Parts:
- added Q1: IRFZ44N, IRFZ44N:TO254P1016X419X2286-3, F.Cu at (176.3, 70.4)
- added R16: R, Resistor_SMD:R_1206_3216Metric, F.Cu at (242.8, 127.6)
- added R17: R, Resistor_SMD:R_1206_3216Metric, F.Cu at (248.4, 127.6)
- added U1: ESP32-DEVKITC-32D, ESP32-WROOM:MODULE_ESP32-WROOM-32, F.Cu at (164.5, 107.2)
- added U3: TCRT5000, QRE1113 IR LED:DIP400W50P180L360H200Q4, F.Cu at (134.2, 61.8)
- added U4: TCRT5000, QRE1113 IR LED:DIP400W50P180L360H200Q4, F.Cu at (266.1, 102.8)
- added U5: TCRT5000, QRE1113 IR LED:DIP400W50P180L360H200Q4, F.Cu at (171.8, 61.8)
- added U6: TCRT5000, QRE1113 IR LED:DIP400W50P180L360H200Q4, F.Cu at (275.2, 102.8)
- added U7: TCRT5000, QRE1113 IR LED:DIP400W50P180L360H200Q4, F.Cu at (146.8, 61.8)
- added U8: TCRT5000, QRE1113 IR LED:DIP400W50P180L360H200Q4, F.Cu at (184.2, 61.8)
- added U9: TCRT5000, QRE1113 IR LED:DIP400W50P180L360H200Q4, F.Cu at (159.2, 61.8)
- moved J1 108.8 mm to (141.2, 143.2), turned to 90 degrees
- moved J2 108.3 mm to (140.9, 147.5), turned to 90 degrees
- moved R18 97.8 mm to (140.5, 60.5)
- moved R5 16.5 mm to (244.5, 94.2)
Routing:
- net (no net): track 0.00 -> 64.8 mm
Other:
- board size 80 x 62.5 mm -> 80.8 x 95 mm
