File: Latest/Latest.kicad_sch (KiCad schematic)
At the start: 57 parts

Commit message: vault backup: 2022-09-11 00:08:13
Parts:
- removed S?: MPB04-2C33-S-D, MPB04-2C33-S-D:SW_MPB04-2C33-S-D, symbol Meshmerize-rescue:MPB04-2C33-S-D-MPB04-2C33-S-D
- Q1: renamed from Q?; footprint TO254P1016X419X2286-3 -> (none)
- U10: renamed from U?; footprint XCVR_ESP32S3WROOM1N8R8 -> (none)
- U11: renamed from U?; footprint XCVR_ESP32-S3-DEVKITC-1-N8R2 -> (none)
- gave numbers to parts that had none: 53
Connections:
- net DEB: no longer names the net of J1.15 (Pin_15), U1.15 (IO13)
- no-connect marks 4 -> 2
Other:
- note added: "Switch"
- note removed: "Debug Switch"
- note removed: "Switches"
- moved on the sheet: S1

Commit message: vault backup: 2022-09-20 17:33:49
Parts:
- R16, R17: footprint (none) -> Resistor_SMD:R_1206_3216Metric
Changed lines of the file:
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@@
     (property "Reference" "R16" (id 0) (at 187.452 146.558 90))
     (property "Value" "R" (id 1) (at 187.198 148.844 90))
-    (property "Footprint" "" (id 2) (at 186.944 152.654 90)
+    (property "Footprint" "Resistor_SMD:R_1206_3216Metric" (id 2) (at 186.944 152.654 90)
       (effects (font (size 1.27 1.27)) hide)
     )
@@
       (effects (font (size 1.27 1.27)) (justify right))
     )
-    (property "Footprint" "" (id 2) (at 193.294 156.972 90)
+    (property "Footprint" "Resistor_SMD:R_1206_3216Metric" (id 2) (at 193.294 156.972 90)
       (effects (font (size 1.27 1.27)) hide)
     )
@@
     )
     (path "/3c872b4d-d368-41c8-bff3-2a878c57d279"
-      (reference "R16") (unit 1) (value "R") (footprint "")
+      (reference "R16") (unit 1) (value "R") (footprint "Resistor_SMD:R_1206_3216Metric")
     )
     (path "/f4df0f64-be65-4a37-96a0-81f0750933fc"
-      (reference "R17") (unit 1) (value "R") (footprint "")
+      (reference "R17") (unit 1) (value "R") (footprint "Resistor_SMD:R_1206_3216Metric")
     )
     (path "/160cf280-bdf9-4f60-9ac9-cb06547dab57"

Commit message: vault backup: 2022-10-02 12:01:12
Parts:
- removed U10: ESP32S3WROOM1N8R8, symbol ESP32S3WROOM1N8R8:ESP32S3WROOM1N8R8
- removed U11: ESP32-S3-DEVKITC-1-N8R2, symbol ESP32-S3-DEVKITC-1-N8R2:ESP32-S3-DEVKITC-1-N8R2
- Q1: footprint (none) -> IRFZ44N:TO254P1016X419X2286-3
- U1: footprint esp32_DEVKITC-32D:MODULE_ESP32-DEVKITC-32D -> ESP32-WROOM:MODULE_ESP32-WROOM-32
- U3, U4, U5, U6, U7, U8, U9: footprint TCRT5000:OPTO_TCRT5000 -> QRE1113 IR LED:DIP400W50P180L360H200Q4
